Commit message: - Cage STL Farbe geben und Glas herum transparent machen. - Candy Colada Fila hinzugefügt - Cage zwischen world_link und base_link hinzugefügt

File: src/msrobot/msrobot_description/urdf/msrobot_follower.urdf.xacro (robot description, xacro)
@@ -12,8 +12,27 @@
     <xacro:include filename="$(find msrobot_description)/urdf/utils.urdf.xacro" />
     <link name="world"></link>
-    <joint name="world_to_base_link" type="fixed">
+    <joint name="world_to_cage" type="fixed">
         <parent link="world" />
+        <child link="cage" />
+        <origin  rpy="0 0 0" xyz="0 0 0" />
+    </joint>
+    <link name="cage">
+        <visual>
+            <origin xyz="0 0 0" rpy="0 0 0"/>
+            <geometry>
+               <mesh filename="package://msrobot_description/meshes/cage/cage.dae" scale="1 1 1"/>
+            </geometry>
+        </visual>
+        <collision>
+            <origin xyz="0 0 0.019" rpy="0 0 0"/>
+            <geometry>
+               <mesh filename="package://msrobot_description/meshes/cage/cage.dae" scale="0 0 0"/>
+            </geometry>
+        </collision>
+    </link>
+    <joint name="cage_to_base_link" type="fixed">
+        <parent link="cage" />
         <child link="base_link" />
-        <origin  rpy="0 0 0" xyz="0 0 0" />
+        <origin xyz="0 0 0.25" rpy="0 0 0"/>
     </joint>
     <link name="base_link">
